Commit message: add librealsense
如果发现topic无法发布realsense信息时，记得拷贝该.so文件至/opt/ros/noetic/lib目录下

File: simulation/src/rotors_simulator/rotors_description/urdf/D435/depthcam.xacro (robot description, xacro)
@@ -225,190 +225,3 @@
     </gazebo>
   </xacro:macro>
-  <!-- INTEL REALSENSE R200 -->
-  <xacro:macro name="realsense_R200" params="sensor_name parent_link rate *origin">
-      <link name="${sensor_name}_R200_camera">
-          <visual>
-              <origin rpy="0 0 0" xyz="0 0 0"/>
-              <geometry>
-                  <mesh filename="package://rotors_description/meshes/realsense_r200/meshes/realsense.dae"/>
-              </geometry>
-          </visual>
-          <collision>
-              <geometry>
-                  <box size="0.0078 0.130 0.0192"/>
-              </geometry>
-          </collision>
-          <inertial>
-              <mass value="0.0615752"/>
-              <origin rpy="0 0 0" xyz="0 0 0"/>
-              <inertia ixx="9.108e-05"
-                       ixy="0"
-                       ixz="0"
-                       iyy="2.51e-06"
-                       iyz="0"
-                       izz="8.931e-05"/>
-          </inertial>
-      </link>
-      <joint name="${sensor_name}_joint" type="fixed">
-          <parent link="${parent_link}"/>
-          <child link="${sensor_name}_R200_camera"/>
-          <xacro:insert_block name="origin"/>
-      </joint>
-      <link name="${sensor_name}_color" />
-      <link name="${sensor_name}_depth" />
-      <link name="${sensor_name}_ired1" />
-      <link name="${sensor_name}_ired2" />
-      <joint name="${sensor_name}_color_joint" type="fixed">
-          <parent link="${sensor_name}_R200_camera" />
-          <child link="${sensor_name}_color" />
-          <origin xyz="0 -0.046 0.004" rpy="${pi/2} ${pi} ${pi/2}"/>
-      </joint>
-      <joint name="${sensor_name}_depth_joint" type="fixed">
-          <parent link="${sensor_name}_R200_camera" />
-          <child link="${sensor_name}_depth" />
-          <origin xyz="0 -0.03 0.004" rpy="0 0 0"/>
-      </joint>
-      <joint name="${sensor_name}_ired1_joint" type="fixed">
-          <parent link="${sensor_name}_R200_camera" />
-          <child link="${sensor_name}_ired1" />
-          <origin xyz="0 -0.06 0.004" rpy="0 0 0"/>
-      </joint>
-      <joint name="${sensor_name}_ired2_joint" type="fixed">
-          <parent link="${sensor_name}_R200_camera" />
-          <child link="${sensor_name}_ired2" />
-          <origin xyz="0 0.01 0.004" rpy="0 0 0"/>
-      </joint>
-      <gazebo reference="${sensor_name}_R200_camera">
-          <self_collide>0</self_collide>
-          <enable_wind>0</enable_wind>
-          <kinematic>0</kinematic>
-          <gravity>1</gravity>
-          <mu>1</mu>
-          <mu2>1</mu2>
-          <fdir1>0 0 0</fdir1>
-          <slip1>0</slip1>
-          <slip2>0</slip2>
-          <kp>1e+13</kp>
-          <kd>1</kd>
-          <max_vel>0.01</max_vel>
-          <min_depth>0</min_depth>
-          <sensor name="${sensor_name}_color" type="camera">
-              <pose frame="">0 -0.046 0.004 0 0 0</pose>
-              <camera name="${sensor_name}_R200_camera">
-              <horizontal_fov>1.047</horizontal_fov>
-              <image>
-                  <width>640</width>
-                  <height>480</height>
-                  <format>RGB_INT8</format>
-              </image>
-              <clip>
-                  <near>0.1</near>
-                  <far>100</far>
-              </clip>
-              <noise>
-                  <type>gaussian</type>
-                  <mean>0.0</mean>
-                  <stddev>0.007</stddev>
-              </noise>
-              </camera>
-              <always_on>1</always_on>
-              <update_rate>${rate}</update_rate>
-              <visualize>1</visualize>
-          </sensor>
-          <sensor name="${sensor_name}_ired1" type="camera">
-              <pose frame="">0 -0.06 0.004 0 0 0</pose>
-              <camera name="${sensor_name}_R200_camera">
-              <horizontal_fov>1.047</horizontal_fov>
-              <image>
-                  <width>640</width>
-                  <height>480</height>
-                  <format>L_INT8</format>
-              </image>
-              <clip>
-                  <near>0.1</near>
-                  <far>100</far>
-              </clip>
-              <noise>
-                  <type>gaussian</type>
-                  <mean>0.0</mean>
-                  <stddev>0.05</stddev>
-              </noise>
-              </camera>
-              <always_on>1</always_on>
-              <update_rate>${rate}</update_rate>
-              <visualize>0</visualize>
-          </sensor>
-          <sensor name="${sensor_name}_ired2" type="camera">
-              <pose frame="">0 0.01 0.004 0 0 0</pose>
-              <camera name="${sensor_name}_R200_camera">
-              <horizontal_fov>1.047</horizontal_fov>
-              <image>
-                  <width>640</width>
-                  <height>480</height>
-                  <format>L_INT8</format>
-              </image>
-              <clip>
-                  <near>0.1</near>
-                  <far>100</far>
-              </clip>
-              <noise>
-                  <type>gaussian</type>
-                  <mean>0.0</mean>
-                  <stddev>0.05</stddev>
-              </noise>
-              </camera>
-              <always_on>1</always_on>
-              <update_rate>${rate}</update_rate>
-              <visualize>0</visualize>
-          </sensor>
-          <sensor name="${sensor_name}_depth" type="depth">
-              <pose frame="">0 -0.03 0.004 0 0 0</pose>
-              <camera name="${sensor_name}_R200_camera">
-              <horizontal_fov>1.047</horizontal_fov>
-              <image>
-                      <width>640</width>
-                      <height>480</height>
-              </image>
-              <clip>
-                      <near>0.1</near>
-                      <far>100</far>
-              </clip>
-              <noise>
-                      <type>gaussian</type>
-                      <mean>0.0</mean>
-                      <stddev>0.100</stddev>
-              </noise>
-              </camera>
-              <always_on>1</always_on>
-              <update_rate>60</update_rate>
-              <visualize>0</visualize>
-          </sensor>
-      </gazebo>
-      <gazebo>
-        <plugin name="${sensor_name}" filename="librealsense_gazebo_plugin.so">
-          <prefix>${sensor_name}_</prefix>
-          <depthUpdateRate>${rate}</depthUpdateRate>
-          <colorUpdateRate>${rate}</colorUpdateRate>
-          <infraredUpdateRate>${rate}</infraredUpdateRate>
-          <depthTopicName>depth/image_raw</depthTopicName>
-          <depthCameraInfoTopicName>depth/camera_info</depthCameraInfoTopicName>
-          <colorTopicName>color/image_raw</colorTopicName>
-          <colorCameraInfoTopicName>color/camera_info</colorCameraInfoTopicName>
-          <infrared1TopicName>infra1/image_raw</infrared1TopicName>
-          <infrared1CameraInfoTopicName>infra1/camera_info</infrared1CameraInfoTopicName>
-          <infrared2TopicName>infra2/image_raw</infrared2TopicName>
-          <infrared2CameraInfoTopicName>infra2/camera_info</infrared2CameraInfoTopicName>
-          <colorOpticalframeName>${sensor_name}_color_optical_frame</colorOpticalframeName>
-          <depthOpticalframeName>${sensor_name}_depth_optical_frame</depthOpticalframeName>
-          <infrared1OpticalframeName>${sensor_name}_infrared1_optical_frame</infrared1OpticalframeName>
-          <infrared2OpticalframeName>${sensor_name}_infrared2_optical_frame</infrared2OpticalframeName>
-          <rangeMinDepth>0.2</rangeMinDepth>
-          <rangeMaxDepth>10.0</rangeMaxDepth>
-          <pointCloud>false</pointCloud>
-          <pointCloudTopicName>depth/color/points</pointCloudTopicName>
-          <pointCloudCutoff>0.25</pointCloudCutoff>
-          <pointCloudCutoffMax>9.0</pointCloudCutoffMax>
-        </plugin>
-      </gazebo>
-  </xacro:macro>
 </robot>
