Commit message: 增加订阅的map_server,添加run.sh一键运行

File: src/simulation/rotors_simulator/rotors_description/urdf/component_snippets.xacro (robot description, xacro)
@@ -739,4 +739,5 @@
         <inertia ixx="0.00001" ixy="0.0" ixz="0.0" iyy="0.00001" iyz="0.0" izz="0.00001" /> <!-- [kg m^2] [kg m^2] [kg m^2] [kg m^2] [kg m^2] [kg m^2] -->
         <origin xyz="0.0 0.0 0.0" rpy="0.0 0.0 0.0" />
+        <!-- <origin xyz="0.1 0.0 -0.03" rpy="0.0 0.27 0.0" /> -->
       </xacro:odometry_plugin_macro>
     </xacro:if>
